Commit message: Node created to monitor IMU sensor

File: balance_bot_description/description/body.xacro (robot description, xacro)
@@ -21,15 +21,7 @@
             </geometry>
         </collision>
-        <inertial>
-            <origin xyz="0 0 ${body_height/2}" />
-            <mass value="${body_mass}" />
-            <inertia
-                ixx="0.05"
-                ixy="0"
-                ixz="0"
-                iyy="0.05"
-                iyz="0"
-                izz="0.01" />
-        </inertial>
+        <xacro:inertial_box mass="${body_mass}" x="${body_depth}" y="${body_width}" z="${body_height}">
+            <origin xyz="0.0 0.0 ${body_height/2}"/>
+        </xacro:inertial_box>
     </link>
 </robot>

File: balance_bot_description/description/bot.urdf.xacro (robot description, xacro)
@@ -4,4 +4,6 @@
     <!-- Colours/Materials -->
     <xacro:include filename="materials.xacro"/>
+    <!-- Inertial properties -->
+    <xacro:include filename="inertial_macros.xacro"/>
     <!-- dimensional constants -->
     <xacro:property name="body_height" value="0.3" />
@@ -12,9 +14,10 @@
     <!-- groud clearance will be same as wheel radius -->
     <xacro:property name="ground_clearance" value="0.05" />
-    <xacro:property name="body_mass" value="2.0" />
-    <xacro:property name="wheel_mass" value="0.2" />
+    <xacro:property name="body_mass" value="1.0" />
+    <xacro:property name="wheel_mass" value="0.1" />
     <!-- Robot Parts -->
     <xacro:include filename="body.xacro"/>
     <xacro:include filename="wheels.xacro"/>
+    <xacro:include filename="imu.xacro"/>
     <!-- Gazebo plugins -->
     <xacro:include filename="gazebo.xacro"/>

File: balance_bot_description/description/gazebo.xacro (robot description, xacro)
@@ -17,3 +17,23 @@
         </plugin>
     </gazebo>
+    <gazebo reference="imu_link">
+        <sensor name="imu_sensor" type="imu">
+            <always_on>true</always_on>
+            <update_rate>200</update_rate>
+            <visualize>true</visualize>
+            <topic>/imu</topic>
+            <imu>
+                <angular_velocity>
+                    <x/>
+                    <y/>
+                    <z/>
+                </angular_velocity>
+                <linear_acceleration>
+                    <x/>
+                    <y/>
+                    <z/>
+                </linear_acceleration>
+            </imu>
+        </sensor>
+    </gazebo>
 </robot>

File: balance_bot_description/description/imu.xacro (robot description, xacro)
@@ -1,3 +1,21 @@
 <?xml version="1.0"?>
 <robot xmlns:xacro="http://www.ros.org/wiki/xacro">
+    <link name="imu_link">
+        <visual>
+            <origin xyz="0 0 0" />
+            <geometry>
+                <box size="0.02 0.02 0.01" />
+            </geometry>
+            <material name="green"></material>
+        </visual>
+        <xacro:inertial_box mass="0.001" x="0.02" y="0.02" z="0.01">
+            <origin xyz="0 0 0"/>
+        </xacro:inertial_box>
+    </link>
+    <joint name="imu_joint" type="fixed">
+        <parent link="body_link" />
+        <child link="imu_link" />
+        <!-- Place IMU near the wheel axle -->
+        <origin xyz="0 0 0" />
+    </joint>
 </robot>

File: balance_bot_description/description/wheels.xacro (robot description, xacro)
@@ -17,14 +17,7 @@
             </geometry>
         </collision>
-        <inertial>
-            <mass value="${wheel_mass}"/>
-            <inertia
-                ixx="0.0003"
-                ixy="0"
-                ixz="0"
-                iyy="0.0003"
-                iyz="0"
-                izz="0.0005"/>
-        </inertial>
+        <xacro:inertial_cylinder mass="${wheel_mass}" radius="${wheel_radius}" length="${wheel_width}">
+            <origin xyz="0 0 0"/>
+        </xacro:inertial_cylinder>
     </link>
     <joint name="left_wheel_joint" type="continuous">
@@ -50,14 +43,7 @@
             </geometry>
         </collision>
-        <inertial>
-            <mass value="${wheel_mass}"/>
-            <inertia
-                ixx="0.0003"
-                ixy="0"
-                ixz="0"
-                iyy="0.0003"
-                iyz="0"
-                izz="0.0005"/>
-        </inertial>
+        <xacro:inertial_cylinder mass="${wheel_mass}" radius="${wheel_radius}" length="${wheel_width}">
+            <origin xyz="0 0 0"/>
+        </xacro:inertial_cylinder>
     </link>
     <joint name="right_wheel_joint" type="continuous">
